File: PWM_Generator_KiCAD/PWM_Generator/PWM_Generator.sch (KiCad schematic (older format))
At the start: 17 parts, among them J1 Screw_Terminal_01x02, J2 Screw_Terminal_01x02, U1 NE555D

Commit message: Add in gerbers
Parts:
- added J3: Screw_Terminal_01x03, Connector_PinHeader_1.00mm:PinHeader_1x03_P1.00mm_Vertical, symbol Connector:Screw_Terminal_01x03
- added TP1, TP2, TP3: TestPoint, TestPoint:TestPoint_Pad_D1.0mm, symbol Connector:TestPoint
- R3: footprint (none) -> KiCADPersonalLibs:P164K101PNN20B103; DIGIKEY_NUM 987-1155-ND -> 987-P164K101PNN20B103-ND
- gave numbers to parts that had none: 2
Connections:
- net GND: now also J3.1 (Pin_1)
- net OUT: now also J3.3 (Pin_3), TP3.1
- net TRIG: now also TP1.1
- net VCC: now also J3.2 (Pin_2)
- net at D2.2 (A), R2.2, R4.1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: now also TP2.1
Other:
- moved on the sheet: C1, C2, C3, C4, D1, D2, D3, D4, J1, J2, Q1, R1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
