File: ESP32_SOIL/soil_sensor/soil_sensor.sch (KiCad schematic (older format))
At the start: 34 parts, among them J1 USB_B_Mini, J2 Screw_Terminal_01x03, J3 Screw_Terminal_01x06, Q1 Q_NPN_BEC, Q2 Q_NPN_BEC, SW1 SW_Push, U1 ESP32-WROOM-32U, U3 LD39015M33R

Commit message: Add in Boost Converter
Parts:
- C1, C2, C3, C4, C5: Digikey (none) -> 311-1824-1-ND
- D1: Digikey (none) -> P14141CT-ND
- D2: Digikey (none) -> 732-4978-1-ND
- D3: Digikey (none) -> 732-4980-1-ND
Changed lines of the file:
@@
 F 2 "Capacitor_SMD:C_0603_1608Metric_Pad1.08x0.95mm_HandSolder" H 2238 6250 50  0001 C CNN
 F 3 "~" H 2200 6400 50  0001 C CNN
+F 4 "311-1824-1-ND" H 2200 6400 50  0001 C CNN "Digikey"
 	1    2200 6400
 	-1   0    0    1
@@
 F 2 "Capacitor_SMD:C_0603_1608Metric_Pad1.08x0.95mm_HandSolder" H 3238 6250 50  0001 C CNN
 F 3 "~" H 3200 6400 50  0001 C CNN
+F 4 "311-1824-1-ND" H 3200 6400 50  0001 C CNN "Digikey"
 	1    3200 6400
 	-1   0    0    1
@@
 F 2 "Capacitor_SMD:C_0603_1608Metric_Pad1.08x0.95mm_HandSolder" H 9738 3200 50  0001 C CNN
 F 3 "~" H 9700 3350 50  0001 C CNN
+F 4 "311-1824-1-ND" H 9700 3350 50  0001 C CNN "Digikey"
 	1    9700 3350
 	-1   0    0    1
@@
 F 2 "Capacitor_SMD:C_0603_1608Metric_Pad1.08x0.95mm_HandSolder" H 8788 1950 50  0001 C CNN
 F 3 "~" H 8750 2100 50  0001 C CNN
+F 4 "311-1824-1-ND" H 8750 2100 50  0001 C CNN "Digikey"
 	1    8750 2100
 	0    1    1    0
@@
 F 2 "LED_SMD:LED_0603_1608Metric_Pad1.05x0.95mm_HandSolder" H 4300 6450 50  0001 C CNN
 F 3 "~" H 4300 6450 50  0001 C CNN
+F 4 "732-4978-1-ND" H 4300 6450 50  0001 C CNN "Digikey"
 	1    4300 6450
 	0    -1   -1   0
@@
 F 2 "LED_SMD:LED_0603_1608Metric_Pad1.05x0.95mm_HandSolder" H 1250 6450 50  0001 C CNN
 F 3 "~" H 1250 6450 50  0001 C CNN
+F 4 "P14141CT-ND" H 1250 6450 50  0001 C CNN "Digikey"
 	1    1250 6450
 	0    -1   -1   0
@@
 F 2 "LED_SMD:LED_0603_1608Metric_Pad1.05x0.95mm_HandSolder" H 9850 4400 50  0001 C CNN
 F 3 "~" H 9850 4400 50  0001 C CNN
+F 4 "732-4980-1-ND" H 9850 4400 50  0001 C CNN "Digikey"
 	1    9850 4400
 	0    -1   -1   0
@@
 F 2 "Capacitor_SMD:C_0603_1608Metric_Pad1.08x0.95mm_HandSolder" H 1738 3050 50  0001 C CNN
 F 3 "~" H 1700 3200 50  0001 C CNN
+F 4 "311-1824-1-ND" H 1700 3200 50  0001 C CNN "Digikey"
 	1    1700 3200
 	-1   0    0    1
