File: CustomESC_KiCAD/CustomESC_KiCAD.kicad_pcb (KiCad board)
At the start: 2 copper layers, 60 parts, among them J1 Screw_Terminal_01x02, J2 Screw_Terminal_01x02, J3 Screw_Terminal_01x06, J4 Screw_Terminal_01x03, J5 Screw_Terminal_01x03, Q1 Q_NMOS_GDS, Q2 Q_NMOS_GDS, Q3 Q_NMOS_GDS, Q4 Q_NMOS_GDS, Q5 Q_NMOS_GDS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

Commit message: Finish Custom ESC layout
Parts:
- added C10: 1nF, Capacitor_SMD:C_0603_1608Metric_Pad1.08x0.95mm_HandSolder, F.Cu at (209.0, 81.8)
- added C11: 1nF, Capacitor_SMD:C_0603_1608Metric_Pad1.08x0.95mm_HandSolder, F.Cu at (199.6, 88.6)
- added C9: 1nF, Capacitor_SMD:C_0603_1608Metric_Pad1.08x0.95mm_HandSolder, F.Cu at (188.0, 81.8)
- added TP4: TestPoint, TestPoint:TestPoint_Pad_D1.0mm, F.Cu at (191.3, 76.2)
- added TP5: TestPoint, TestPoint:TestPoint_Pad_D1.0mm, F.Cu at (205.7, 79.0)
- added TP6: TestPoint, TestPoint:TestPoint_Pad_D1.0mm, F.Cu at (196.6, 86.4)
- J2: footprint TerminalBlock_Phoenix:TerminalBlock_Phoenix_MKDS-1,5-2_1x02_P5.00mm_Horizontal -> Connector_PinHeader_2.54mm:PinHeader_1x02_P2.54mm_Vertical
- J5: value Screw_Terminal_01x03 -> Screw_Terminal_01x04; footprint Connector_PinHeader_2.54mm:PinHeader_1x03_P2.54mm_Vertical -> Connector_PinHeader_2.54mm:PinHeader_1x04_P2.54mm_Vertical
- Q2, Q4, Q6: moved to B.Cu
- moved R28 72.3 mm to (206.0, 72.4), turned to 270 degrees
- moved U4 71.8 mm to (198.5, 76.3)
- moved R18 71.1 mm to (209.1, 76.5)
- moved R27 69.7 mm to (189.0, 72.4), turned to 270 degrees
- moved R21 69.6 mm to (209.0, 79.8)
- moved R24 68.9 mm to (205.2, 76.5)
- moved R17 67.3 mm to (188.0, 78.7), turned to 180 degrees
- moved R26 67.0 mm to (192.3, 72.4), turned to 270 degrees
- moved R20 65.3 mm to (188.0, 75.7), turned to 180 degrees
- moved R19 65.1 mm to (199.6, 83.6)
- moved R22 63.6 mm to (199.6, 86.6)
- moved R25 62.9 mm to (195.8, 83.6)
- moved R23 60.1 mm to (192.0, 78.7), turned to 180 degrees
- moved C8 57.9 mm to (199.4, 58.7), turned to 270 degrees
- moved D1 47.7 mm to (208.8, 59.7), turned to 90 degrees
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Connections:
- R4 pad 1: VBUS -> VCC
Routing:
- net VBUS: track 0.00 -> 137.8 mm, vias 0 -> 18
- net PHASEA: track 0.00 -> 68.5 mm, vias 0 -> 2
- net /OD_A: track 0.00 -> 62.8 mm, vias 0 -> 2
- net /IN_A: track 0.00 -> 58.5 mm, vias 0 -> 2
- net NEUT: track 0.00 -> 48.0 mm, vias 0 -> 1
- net /OD_B: track 0.00 -> 43.5 mm, vias 0 -> 2
- net ZCROSS_A: track 0.00 -> 40.5 mm, vias 0 -> 1
- net /BackEMF/BEMFB: track 0.00 -> 40.2 mm, vias 0 -> 4
- net /IN_B: track 0.00 -> 39.5 mm, vias 0 -> 2
- net ZCROSS_B: track 0.00 -> 38.8 mm, vias 0 -> 1
- net PHASEC: track 0.00 -> 38.3 mm, vias 0 -> 2
- net ZCROSS_C: track 0.00 -> 35.4 mm, vias 0 -> 1
- net /OD_C: track 0.00 -> 33.7 mm, vias 0 -> 1
- net GND: track 0.00 -> 32.2 mm, vias 0 -> 9
- net PHASEB: track 0.00 -> 29.3 mm, vias 0 -> 2
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- added copper zone on F.Cu, net GND
- added copper zone on In1.Cu, net GND
- added copper zone on B.Cu, net PHASEA
- added copper zone on F.Cu, net PHASEA
- added copper zone on B.Cu, net PHASEB
- added copper zone on F.Cu, net PHASEB
- added copper zone on B.Cu, net PHASEC
- added copper zone on F.Cu, net PHASEC
- added copper zone on F.Cu, net VBUS
- added copper zone on In2.Cu, net VBUS
- added copper zone on In2.Cu, net VCC
Other:
- board outline added: 80 x 53.3 mm
- copper layers 2 -> 4
- board text added: "+ (12V)"
- board text added: "+ -"
- board text added: "-"
- board text added: "CABBAGES!!"
- board text added: "NEUT"
- board text added: "OD_A IN_A"
- board text added: "OD_B IN_B"
- board text added: "OD_C IN_C"
- board text added: "Sensorless ESC Sahil Kale 10/23/2021"
- board text added: "ZA ZB ZC"
