File: CustomESC_KiCAD/CustomESC_KiCAD.kicad_pcb (KiCad board)
At the start: 4 copper layers, 80 x 53.3 mm, 66 parts, among them J1 Screw_Terminal_01x02, J2 Screw_Terminal_01x02, J3 Screw_Terminal_01x06, J4 Screw_Terminal_01x03, J5 Screw_Terminal_01x04, Q1 Q_NMOS_GDS, Q2 Q_NMOS_GDS, Q3 Q_NMOS_GDS, Q4 Q_NMOS_GDS, Q5 Q_NMOS_GDS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

Commit message: random stuff for custom esc
Other:
- net class Default removed
