File: CustomESC_KiCAD/_autosave-BackEMF.sch (KiCad schematic (older format))
At the start: 19 parts, among them U4 LM339

Commit message: Finish Custom ESC layout
Parts:
- removed C?: 1nF, symbol Device:C_Small
- added C9: 1nF, Capacitor_SMD:C_0603_1608Metric_Pad1.08x0.95mm_HandSolder, symbol Device:C_Small
- C10, C11: renamed from C?; footprint (none) -> Capacitor_SMD:C_0603_1608Metric_Pad1.08x0.95mm_HandSolder; Digikey Number (none) -> 399-17878-1-ND
Connections:
- net BEMFA: now also C9.1
- net GND: now also C9.2
Changed lines of the file:
@@
 	6000 3950 6750 3950
 $Comp
-L Device:C_Small C?
-U 1 1 617F6620
-P 5850 2850
-F 0 "C?" H 5942 2896 50  0000 L CNN
-F 1 "1nF" H 5942 2805 50  0000 L CNN
-F 2 "" H 5850 2850 50  0001 C CNN
-F 3 "~" H 5850 2850 50  0001 C CNN
-	1    5850 2850
-	1    0    0    -1
-$EndComp
-$Comp
-L Device:C_Small C?
+L Device:C_Small C10
 U 1 1 617F77EE
 P 5850 3500
-F 0 "C?" H 5942 3546 50  0000 L CNN
+F 0 "C10" H 5942 3546 50  0000 L CNN
 F 1 "1nF" H 5942 3455 50  0000 L CNN
-F 2 "" H 5850 3500 50  0001 C CNN
+F 2 "Capacitor_SMD:C_0603_1608Metric_Pad1.08x0.95mm_HandSolder" H 5850 3500 50  0001 C CNN
 F 3 "~" H 5850 3500 50  0001 C CNN
+F 4 "399-17878-1-ND" H 5850 3500 50  0001 C CNN "Digikey Number"
 	1    5850 3500
 	1    0    0    -1
 $EndComp
 $Comp
-L Device:C_Small C?
+L Device:C_Small C11
 U 1 1 617F7DE6
 P 5850 4100
-F 0 "C?" H 5942 4146 50  0000 L CNN
+F 0 "C11" H 5942 4146 50  0000 L CNN
 F 1 "1nF" H 5942 4055 50  0000 L CNN
-F 2 "" H 5850 4100 50  0001 C CNN
+F 2 "Capacitor_SMD:C_0603_1608Metric_Pad1.08x0.95mm_HandSolder" H 5850 4100 50  0001 C CNN
 F 3 "~" H 5850 4100 50  0001 C CNN
+F 4 "399-17878-1-ND" H 5850 4100 50  0001 C CNN "Digikey Number"
 	1    5850 4100
 	1    0    0    -1
@@
 	5850 3350 6000 3350
 Connection ~ 6000 3350
-Wire Wire Line
-	5850 2750 6000 2750
-Connection ~ 6000 2750
 $Comp
-L power:GND #PWR?
+L power:GND #PWR0103
 U 1 1 61802A49
 P 5850 4200
-F 0 "#PWR?" H 5850 3950 50  0001 C CNN
+F 0 "#PWR0103" H 5850 3950 50  0001 C CNN
 F 1 "GND" H 5855 4027 50  0000 C CNN
 F 2 "" H 5850 4200 50  0001 C CNN
@@
 $EndComp
 $Comp
-L power:GND #PWR?
+L power:GND #PWR0104
 U 1 1 6180313E
 P 5850 3600
-F 0 "#PWR?" H 5850 3350 50  0001 C CNN
+F 0 "#PWR0104" H 5850 3350 50  0001 C CNN
 F 1 "GND" H 5855 3427 50  0000 C CNN
 F 2 "" H 5850 3600 50  0001 C CNN
@@
 $EndComp
 $Comp
-L power:GND #PWR?
+L power:GND #PWR0105
 U 1 1 61803753
-P 5850 2950
-F 0 "#PWR?" H 5850 2700 50  0001 C CNN
-F 1 "GND" H 5855 2777 50  0000 C CNN
-F 2 "" H 5850 2950 50  0001 C CNN
-F 3 "" H 5850 2950 50  0001 C CNN
-	1    5850 2950
+P 5850 3000
+F 0 "#PWR0105" H 5850 2750 50  0001 C CNN
+F 1 "GND" H 5855 2827 50  0000 C CNN
+F 2 "" H 5850 3000 50  0001 C CNN
+F 3 "" H 5850 3000 50  0001 C CNN
+	1    5850 3000
 	1    0    0    -1
 $EndComp
+$Comp
+L Device:C_Small C9
+U 1 1 618072A2
+P 5850 2900
+F 0 "C9" H 5942 2946 50  0000 L CNN
+F 1 "1nF" H 5942 2855 50  0000 L CNN
+F 2 "Capacitor_SMD:C_0603_1608Metric_Pad1.08x0.95mm_HandSolder" H 5850 2900 50  0001 C CNN
+F 3 "~" H 5850 2900 50  0001 C CNN
+F 4 "399-17878-1-ND" H 5850 2900 50  0001 C CNN "Digikey Number"
+	1    5850 2900
+	1    0    0    -1
+$EndComp
+Wire Wire Line
+	6000 2750 5850 2750
+Wire Wire Line
+	5850 2750 5850 2800
+Connection ~ 6000 2750
 $EndSCHEMATC
