File: Joystick/joystick/LCD.kicad_sch (KiCad schematic)
At the start: 3 parts, among them U2 NHD-C0220BIZ

Commit message: Update joystick files
Other:
- company: (none) -> AUTHOR: Sahil Kale
- title: (none) -> Liquid Crystal Display
Changed lines of the file:
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@@
 (kicad_sch (version 20211123) (generator eeschema)
   (paper "A4")
+  (title_block
+    (title "Liquid Crystal Display")
+    (date "2022-08-27")
+    (rev "1.0")
+    (company "AUTHOR: Sahil Kale")
+  )
   (junction (at 158.75 87.63) (diameter 0) (color 0 0 0 0)
   )
