File: Joystick/joystick/MCU.kicad_sch (KiCad schematic)
At the start: 11 parts, among them J6 PROG HEADER, U3 KC2520Z24, U4 STM32L151CBTx

Commit message: Update joystick files
Parts:
- added C18, C19, C20, C21, C22: 0.1uF, Capacitor_SMD:C_0603_1608Metric_Pad1.08x0.95mm_HandSolder, symbol Device:C_Small
Connections:
- net +3V3: now also C18.1, C19.1, C20.1, C21.1, C22.1
- net GND: now also C18.2, C19.2, C20.2, C21.2, C22.2
Other:
- company: (none) -> AUTHOR: Sahil Kale
- title: (none) -> Microcontroller
- moved on the sheet: J6, R11, R12, TP3, TP4, TP5, TP6, TP7, TP8, U3, U4
