File: Joystick/joystick/analog.kicad_sch (KiCad schematic)
At the start: 6 parts, among them U1 ADS130B04

Commit message: Update joystick files
Other:
- company: (none) -> AUTHOR: Sahil Kale
- title: (none) -> Analog to Digital Converter
Changed lines of the file:
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@@
 (kicad_sch (version 20211123) (generator eeschema)
   (paper "A4")
+  (title_block
+    (title "Analog to Digital Converter")
+    (date "2022-08-27")
+    (rev "1.0")
+    (company "AUTHOR: Sahil Kale")
+  )
   (junction (at 129.54 91.44) (diameter 0) (color 0 0 0 0)
   )
