File: Joystick/joystick/button_interfaces.kicad_sch.kicad_sch (KiCad schematic)
At the start: 21 parts, among them SW1 SW_Push, SW2 SW_Push, SW3 SW_Push, SW4 SW_Push, SW5 SW_Push, SW6 SW_Push

Commit message: Update joystick files
Parts:
- gave numbers to parts that had none: 3
Other:
- company: (none) -> AUTHOR: Sahil Kale
- title: (none) -> Button Interfaces
Changed lines of the file:
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@@
 (kicad_sch (version 20211123) (generator eeschema)
   (paper "A4")
+  (title_block
+    (title "Button Interfaces")
+    (date "2022-08-27")
+    (rev "1.0")
+    (company "AUTHOR: Sahil Kale")
+  )
   (junction (at 176.53 128.27) (diameter 0) (color 0 0 0 0)
   )
@@
   (symbol (lib_id "Device:R_US") (at 180.34 123.19 0) (unit 1)
     (in_bom yes) (on_board yes) (fields_autoplaced)
-    (property "Reference" "R?" (id 0) (at 181.991 122.2815 0)
+    (property "Reference" "R14" (id 0) (at 181.991 122.2815 0)
       (effects (font (size 1.27 1.27)) (justify left))
     )
@@
   (symbol (lib_id "Device:C_Small") (at 176.53 134.62 0) (unit 1)
     (in_bom yes) (on_board yes)
-    (property "Reference" "C?" (id 0) (at 171.45 133.35 0))
+    (property "Reference" "C4" (id 0) (at 171.45 133.35 0))
     (property "Value" "10nF" (id 1) (at 171.45 135.89 0))
     (property "Footprint" "Capacitor_SMD:C_0603_1608Metric_Pad1.08x0.95mm_HandSolder" (id 2) (at 176.53 134.62 0)
@@
   (symbol (lib_id "power:+3V3") (at 180.34 118.11 0) (unit 1)
     (in_bom yes) (on_board yes) (fields_autoplaced)
-    (property "Reference" "#PWR?" (id 0) (at 180.34 121.92 0)
+    (property "Reference" "#PWR0123" (id 0) (at 180.34 121.92 0)
       (effects (font (size 1.27 1.27)) hide)
     )
@@
   (symbol (lib_id "Switch:SW_Push") (at 180.34 134.62 270) (unit 1)
     (in_bom yes) (on_board yes) (fields_autoplaced)
-    (property "Reference" "SW?" (id 0) (at 184.023 133.7115 90)
+    (property "Reference" "SW7" (id 0) (at 184.023 133.7115 90)
       (effects (font (size 1.27 1.27)) (justify left))
     )
@@
   (symbol (lib_id "power:GND") (at 180.34 142.24 0) (unit 1)
     (in_bom yes) (on_board yes) (fields_autoplaced)
-    (property "Reference" "#PWR?" (id 0) (at 180.34 148.59 0)
-      (effects (font (size 1.27 1.27)) hide)
-    )
+    (property "Reference" "#PWR0124" (id 0) (at 180.34 148.59 0)
+      (effects (font (size 1.27 1.27)) hide)
+    )
