File: Joystick/joystick/joystick.kicad_pcb (KiCad board)
At the start: 2 copper layers, 57 parts, among them J1 Conn_01x03_Male, J2 Conn_01x03_Male, J3 Conn_01x03_Male, J4 Conn_01x03_Male, J5 USB_C_Receptacle_USB2.0, J6 PROG HEADER, SW1 SW_Push, SW2 SW_Push, SW3 SW_Push, SW4 SW_Push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

Commit message: Update joystick files
Parts:
- added C18: 0.1uF, Capacitor_SMD:C_0603_1608Metric_Pad1.08x0.95mm_HandSolder, F.Cu at (178.5, 72.0)
- added C19: 0.1uF, Capacitor_SMD:C_0603_1608Metric_Pad1.08x0.95mm_HandSolder, F.Cu at (189.6, 72.9)
- added C20: 0.1uF, Capacitor_SMD:C_0603_1608Metric_Pad1.08x0.95mm_HandSolder, F.Cu at (177.9, 80.6)
- added C21: 0.1uF, Capacitor_SMD:C_0603_1608Metric_Pad1.08x0.95mm_HandSolder, F.Cu at (190.6, 78.5)
- added C22: 0.1uF, Capacitor_SMD:C_0603_1608Metric_Pad1.08x0.95mm_HandSolder, F.Cu at (188.5, 81.0)
- added H1: MountingHole, MountingHole:MountingHole_2.1mm, F.Cu at (143.3, 72.5)
- added H2: MountingHole, MountingHole:MountingHole_2.1mm, F.Cu at (195.5, 72.0)
- added H4: MountingHole, MountingHole:MountingHole_2.1mm, F.Cu at (195.5, 90.0)
- added R14: 5.1k, Resistor_SMD:R_0603_1608Metric_Pad0.98x0.95mm_HandSolder, F.Cu at (168.5, 84.0)
- added SW7: SW_Push, Button_Switch_SMD:SW_Push_1P1T_NO_6x6mm_H9.5mm, F.Cu at (172.0, 90.5)
- C4: value 1uF -> 10nF
- moved C15 131.6 mm to (215.4, 54.8)
- moved U6 126.0 mm to (215.1, 57.4)
- moved J4 125.3 mm to (216.5, 85.8)
- moved D1 124.6 mm to (214.0, 62.0), turned to 180 degrees
- moved C14 123.8 mm to (212.0, 57.7), turned to -90 degrees
- moved J3 120.6 mm to (216.5, 77.0)
- moved C13 118.2 mm to (206.9, 57.7), turned to -90 degrees
- moved U5 117.5 mm to (209.4, 58.0)
- moved C16 116.9 mm to (209.4, 55.7), turned to 180 degrees
- moved C17 116.5 mm to (214.9, 59.9)
- moved R13 115.2 mm to (210.5, 62.0)
- moved C1 82.8 mm to (159.5, 77.0), turned to 90 degrees
- moved U1 80.5 mm to (154.6, 79.8)
- moved C11 75.6 mm to (167.2, 70.4)
- moved C3 75.3 mm to (156.7, 75.5), turned to 180 degrees
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Connections:
- net /MCU/D+ renamed /USB/D+
- net /MCU/D- renamed /USB/D-
- C4 pad 1: +5V -> /Button Interfaces/USER_SW_3
- TP7 pad 1: /Analog Interfaces/MOSI -> /Analog Interfaces/MISO
- TP8 pad 1: /Analog Interfaces/MISO -> /Analog Interfaces/MOSI
- U4 pad 16: /Analog Interfaces/MOSI -> /Analog Interfaces/MISO
- U4 pad 17: /Analog Interfaces/MISO -> /Analog Interfaces/MOSI
- U4 pad 21: /SW_3 -> /Button Interfaces/SW_3
- U4 pad 22: /SW_4 -> /Button Interfaces/SW_4
- U4 pad 25: /USER_SW_1 -> /Button Interfaces/USER_SW_1
- U4 pad 26: /USER_SW_2 -> /Button Interfaces/USER_SW_2
- U4 pad 27: unconnected-(U4-Pad27) -> /Button Interfaces/USER_SW_3
- U4 pad 45: /SW_1 -> /Button Interfaces/SW_1
- U4 pad 46: /SW_2 -> /Button Interfaces/SW_2
Routing:
- net +1V2: track 0.00 -> 170.4 mm, vias 0 -> 2
- net /USB/D+: track 0.00 -> 84.8 mm, vias 0 -> 2
- net /USB/D-: track 0.00 -> 84.4 mm, vias 0 -> 2
- net /Analog Interfaces/AIN2: track 0.00 -> 79.0 mm, vias 0 -> 1
- net /Button Interfaces/SW_2: track 0.00 -> 76.1 mm, vias 0 -> 2
- net /Analog Interfaces/AIN3: track 0.00 -> 74.1 mm, vias 0 -> 1
- net /Button Interfaces/SW_1: track 0.00 -> 70.3 mm, vias 0 -> 4
- net +3V3: track 0.00 -> 64.6 mm, vias 0 -> 17
- net GND: track 0.00 -> 60.9 mm, vias 0 -> 9
- net /Button Interfaces/SW_3: track 0.00 -> 55.5 mm, vias 0 -> 2
- net /Button Interfaces/SW_4: track 0.00 -> 50.2 mm
- net /Button Interfaces/USER_SW_1: track 0.00 -> 49.4 mm, vias 0 -> 2
- net /Analog Interfaces/CS: track 0.00 -> 44.1 mm, vias 0 -> 2
- net /Analog Interfaces/SCLK: track 0.00 -> 42.4 mm, vias 0 -> 2
- net /Button Interfaces/USER_SW_3: track 0.00 -> 42.2 mm, vias 0 -> 2
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- added copper zone on In2.Cu, net +3V3
- added copper zone on B.Cu, net GND
- added copper zone on F.Cu, net GND
- added copper zone on In1.Cu, net GND
Other:
- board outline added: 92 x 59 mm
- copper layers 2 -> 4
- board text added: "->"
- board text added: "1"
- board text added: "2"
- board text added: "3"
- board text added: "4"
- board text added: "<-"
- board text added: "ENTER"
- board text added: "Robotic HID"
- board text added: "Robotic Human Interface Device Sahil Kale Rev 1.0 6/20/2022"
