File: Joystick/joystick/joystick.kicad_sch (KiCad schematic)
At the start: 0 parts

Commit message: Update joystick files
Other:
- added sheet Mounting Holes (Mounting.kicad_sch)
- company: (none) -> AUTHOR: Sahil Kale
- title: (none) -> COVER
