File: Joystick/joystick/joystick_conn.kicad_sch (KiCad schematic)
At the start: 4 parts, among them J1 Conn_01x03_Male, J2 Conn_01x03_Male, J3 Conn_01x03_Male, J4 Conn_01x03_Male

Commit message: Update joystick files
Other:
- company: (none) -> AUTHOR: Sahil Kale
Changed lines of the file:
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@@
 (kicad_sch (version 20211123) (generator eeschema)
   (paper "A4")
+  (title_block
+    (date "2022-08-27")
+    (rev "1.0")
+    (company "AUTHOR: Sahil Kale")
+  )
   (wire (pts (xy 133.35 114.3) (xy 130.81 114.3))
     (stroke (width 0) (type default) (color 0 0 0 0))
