File: Joystick/joystick/regulators.kicad_sch (KiCad schematic)
At the start: 9 parts, among them U5 MIC5365-3.3YC5, U6 ISL6002DIH

Commit message: Update joystick files
Other:
- company: (none) -> AUTHOR: Sahil Kale
- title: (none) -> Regulators
Changed lines of the file:
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@@
 (kicad_sch (version 20211123) (generator eeschema)
   (paper "A4")
+  (title_block
+    (title "Regulators")
+    (date "2022-08-27")
+    (rev "1.0")
+    (company "AUTHOR: Sahil Kale")
+  )
   (junction (at 102.87 73.66) (diameter 0) (color 0 0 0 0)
   )
