File: Joystick/joystick/usbc.kicad_sch (KiCad schematic)
At the start: 5 parts, among them J5 USB_C_Receptacle_USB2.0

Commit message: Update joystick files
Other:
- company: (none) -> AUTHOR: Sahil Kale
- title: (none) -> USB Interface
Changed lines of the file:
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@@
 (kicad_sch (version 20211123) (generator eeschema)
   (paper "A4")
+  (title_block
+    (title "USB Interface")
+    (date "2022-08-27")
+    (rev "1.0")
+    (company "AUTHOR: Sahil Kale")
+  )
   (junction (at 133.35 95.25) (diameter 0) (color 0 0 0 0)
   )
@@
     (stroke (width 0) (type default) (color 0 0 0 0))
   )
+  (label "D-" (at 156.21 90.17 0)
+    (effects (font (size 1.27 1.27)) (justify left bottom))
+  )
+  (label "D+" (at 156.21 95.25 0)
+    (effects (font (size 1.27 1.27)) (justify left bottom))
+  )
   (hierarchical_label "D+" (shape bidirectional) (at 163.83 95.25 0)
